File: PCB/AM/AM.kicad_sch (KiCad schematic)
At the start: 8 parts, among them J4 Conn_01x05

Commit message: Cleaning, schematics and POC 5
Parts:
- J4: footprint (none) -> Connector_PinHeader_2.54mm:PinHeader_1x05_P2.54mm_Vertical
- S1: footprint (none) -> Connector_PinHeader_2.54mm:PinHeader_1x02_P2.54mm_Vertical
Other:
- company: (none) -> DIKU Design
- title: (none) -> Air Module
- moved on the sheet: D1, D2, J4, R1, R2, S1, S2, Sensor
