File: PCB/AM/AM.kicad_pcb (KiCad board)
At the start: 2 copper layers, 30.5 x 30.5 mm, 10 parts, among them J4 Conn_01x05

Commit message: Some progress
Other:
- board text added: "Air Module"
- board text removed: "Air Module DIKU Design Use with {dblquote}Base Module - Air{dblquote}"
Changed lines of the file:
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@@
       (outputformat 1)
       (mirror false)
-      (drillshape 1)
+      (drillshape 0)
       (scaleselection 1)
-      (outputdirectory "")
+      (outputdirectory "../AM_Gerber/")
     )
   )
@@
     (fp_circle (center 0 0) (end 3.2 0) (layer "Cmts.User") (width 0.15) (fill none))
     (fp_circle (center 0 0) (end 3.45 0) (layer "F.CrtYd") (width 0.05) (fill none))
-    (pad "" np_thru_hole circle (at 0 0) (size 3.2 3.2) (drill 3.2) (layers *.Cu *.Mask))
+    (pad "" thru_hole circle (at 0 0) (size 3.2 3.2) (drill 3.2) (layers *.Cu *.Mask))
   )
   (footprint "LED_THT:LED_D5.0mm" (layer "F.Cu")
@@
     (fp_circle (center 0 0) (end 3.2 0) (layer "Cmts.User") (width 0.15) (fill none))
     (fp_circle (center 0 0) (end 3.45 0) (layer "F.CrtYd") (width 0.05) (fill none))
-    (pad "" np_thru_hole circle (at 0 0) (size 3.2 3.2) (drill 3.2) (layers F&B.Cu *.Mask))
+    (pad "" thru_hole circle (at 0 0) (size 3.2 3.2) (drill 3.2) (layers *.Cu *.Mask))
   )
   (footprint "Connector_PinHeader_2.54mm:PinHeader_1x04_P2.54mm_Vertical" (layer "F.Cu")
@@
     (effects (font (size 1 0.9) (thickness 0.15)))
   )
-  (gr_text "Air Module\nDIKU Design\nUse with {dblquote}Base \nModule - Air{dblquote}\n" (at 175.26 85.09) (layer "F.SilkS")
+  (gr_text "Air Module" (at 175.26 81.28) (layer "F.SilkS")
     (effects (font (size 1 0.9) (thickness 0.15)) (justify left))
   )

Commit message: Cleaning, schematics and POC 5
Changed lines of the file:
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@@
     (tags "mounting hole 3.2mm no annular m3")
     (attr exclude_from_pos_files exclude_from_bom)
-    (fp_text reference "H2" (at 5.08 0) (layer "F.SilkS")
+    (fp_text reference "H2" (at 0 5.08) (layer "F.SilkS")
       (effects (font (size 1 1) (thickness 0.15)))
     )
@@
     (fp_circle (center 0 0) (end 3.2 0) (layer "Cmts.User") (width 0.15) (fill none))
     (fp_circle (center 0 0) (end 3.45 0) (layer "F.CrtYd") (width 0.05) (fill none))
-    (pad "" thru_hole circle (at 0 0) (size 3.2 3.2) (drill 3.2) (layers *.Cu *.Mask))
+    (pad "" np_thru_hole circle (at 0 0) (size 3.2 3.2) (drill 3.2) (layers F&B.Cu *.Mask))
   )
   (footprint "LED_THT:LED_D5.0mm" (layer "F.Cu")
@@
       (effects (font (size 1 1) (thickness 0.15)))
     )
-    (fp_text value "MountingHole_3.2mm_M3" (at 0 4.2) (layer "F.Fab")
+    (fp_text value "MountingHole_3.2mm_M3" (at 0 4.2) (layer "F.Fab") hide
       (effects (font (size 1 1) (thickness 0.15)))
     )
@@
     (fp_circle (center 0 0) (end 3.2 0) (layer "Cmts.User") (width 0.15) (fill none))
     (fp_circle (center 0 0) (end 3.45 0) (layer "F.CrtYd") (width 0.05) (fill none))
-    (pad "" thru_hole circle (at 0 0) (size 3.2 3.2) (drill 3.2) (layers *.Cu *.Mask))
+    (pad "" np_thru_hole circle (at 0 0) (size 3.2 3.2) (drill 3.2) (layers *.Cu *.Mask))
   )
   (footprint "Connector_PinHeader_2.54mm:PinHeader_1x04_P2.54mm_Vertical" (layer "F.Cu")
@@
       (effects (font (size 1 1) (thickness 0.15)))
     )
-    (fp_text value "Conn_01x02" (at 0 4.87) (layer "F.Fab")
-      (effects (font (size 1 1) (thickness 0.15)))
-    )
+    (fp_text value "Conn_01x02" (at 0 4.87) (layer "F.Fab") hide
+      (effects (font (size 1 1) (thickness 0.15)))
+    )

Commit message: Flere billedere
Parts:
- moved D1 102.9 mm to (69.8, 93.3)
- moved D2 102.9 mm to (69.8, 101.6)
- moved H1 102.9 mm to (62.2, 80.0)
- moved H2 102.9 mm to (87.6, 105.4)
- moved J4 102.9 mm to (87.6, 80.0)
- moved S1 102.9 mm to (62.2, 93.3)
- moved S2 102.9 mm to (62.2, 101.6)
- moved Sensor 102.9 mm to (67.3, 80.0)
- moved R1 102.9 mm to (76.2, 93.3)
- moved R2 102.9 mm to (76.2, 101.6)
